File: design/STGSv0.2.kicad_sch (KiCad schematic)
At the start: 56 parts, among them J1 USB_B, J2 DC_Barrel_Jack, J3 AVR-ISP-6, J4 9V-OUT, J5 9V-OUT, J6 5V-OUT, J7 5V-OUT, J8 USB_A_Male, Q1 FDN340P, Q2 DTD113Z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

Commit message: Add files via upload
Other:
- note added: "R5 = 150 R1 = 100k Adjusted for application, to waste less power and shorter on time"
Changed lines of the file:
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@@
     (effects (font (size 1.27 1.27)) (justify left bottom))
   )
-  (text "I=U/R, 5v/33= 150mA" (at 232.41 40.64 0)
+  (text "I=U/R, 5v/33= 150mA" (at 232.41 45.72 0)
     (effects (font (size 2 2) (thickness 0.254) bold) (justify right bottom))
   )
@@
     (effects (font (size 3 3) bold) (justify left bottom))
   )
-  (text "150mA load for PB" (at 232.41 36.83 0)
+  (text "150mA load for PB" (at 228.6 41.91 0)
     (effects (font (size 2 2) (thickness 0.254) bold) (justify right bottom))
   )
@@
     (effects (font (size 1.27 1.27)) (justify left bottom))
   )
+  (text "R5 = 150 \nR1 = 100k \nAdjusted for application, \nto waste less power and shorter on time "
+    (at 194.31 34.29 0)
+    (effects (font (size 1.27 1.27) (color 255 0 0 1)) (justify left bottom))
+  )
   (text "470mV, 3A" (at 265.43 71.12 0)
